Commit message: s

File: body.urdf (robot description, URDF)
Before this commit: robot robot, 3 links, 2 joints
Links:
- added link LeftLeg, mass 1; collision box size=1 0.2 0.2; visual box size=1 0.2 0.2
- link BackLeg: geometry collision box size=0.2 1 0.2; visual box size=0.2 1 0.2
- link FrontLeg: geometry collision box size=0.2 1 0.2; visual box size=0.2 1 0.2
Joints:
- added joint Torso_LeftLeg: type revolute, parent Torso, child LeftLeg, origin xyz=-0.5 0 1 rpy=0 0 0, axis 1 0 0, limit lower=-3.14159 upper=3.14159 effort=0.0 velocity=0.0
- joint Torso_BackLeg: axis 0 1 0 -> 1 0 0; origin xyz=1 0 1 rpy=0 0 0 -> xyz=0 -0.5 1 rpy=0 0 0
- joint Torso_FrontLeg: axis 0 1 0 -> 1 0 0; origin xyz=2 0 1 rpy=0 0 0 -> xyz=0 0.5 1 rpy=0 0 0

Commit message: quadruped

File: body.urdf (robot description, URDF)
Before this commit: robot robot, 4 links, 3 joints
Links:
- added link LowerBackLeg, mass 1; collision box size=0.2 0.2 1; visual box size=0.2 0.2 1
- added link LowerFrontLeg, mass 1; collision box size=0.2 0.2 1; visual box size=0.2 0.2 1
- added link LowerLeftLeg, mass 1; collision box size=0.2 0.2 1; visual box size=0.2 0.2 1
- added link LowerRightLeg, mass 1; collision box size=0.2 0.2 1; visual box size=0.2 0.2 1
- added link RightLeg, mass 1; collision box size=1 0.2 0.2; visual box size=1 0.2 0.2
Joints:
- added joint BackLeg_LowerBackLeg: type revolute, parent BackLeg, child LowerBackLeg, origin xyz=0 -1 0 rpy=0 0 0, axis 1 0 0, limit lower=-3.14159 upper=3.14159 effort=0.0 velocity=0.0
- added joint FrontLeg_LowerFrontLeg: type revolute, parent FrontLeg, child LowerFrontLeg, origin xyz=0 1 0 rpy=0 0 0, axis 1 0 0, limit lower=-3.14159 upper=3.14159 effort=0.0 velocity=0.0
- added joint LeftLeg_LowerLeftLeg: type revolute, parent LeftLeg, child LowerLeftLeg, origin xyz=-1 0 0 rpy=0 0 0, axis 0 1 0, limit lower=-3.14159 upper=3.14159 effort=0.0 velocity=0.0
- added joint RightLeg_LowerRightLeg: type revolute, parent RightLeg, child LowerRightLeg, origin xyz=1 0 0 rpy=0 0 0, axis 0 1 0, limit lower=-3.14159 upper=3.14159 effort=0.0 velocity=0.0
- added joint Torso_RightLeg: type revolute, parent Torso, child RightLeg, origin xyz=0.5 0 1 rpy=0 0 0, axis 0 1 0, limit lower=-3.14159 upper=3.14159 effort=0.0 velocity=0.0
- joint Torso_LeftLeg: axis 1 0 0 -> 0 1 0

Commit message: snake without brain

File: body.urdf (robot description, URDF)
Before this commit: robot robot, 9 links, 8 joints
Links:
- removed link BackLeg
- removed link FrontLeg
- removed link LeftLeg
- removed link LowerBackLeg
- removed link LowerFrontLeg
- removed link LowerLeftLeg
- removed link LowerRightLeg
- removed link RightLeg
- removed link Torso
- added link Link0, mass 1; collision box size=0.6943004632299414 0.8907047373314598 0.9248489599531136; visual box size=0.6943004632299414 0.8907047373314598 0.9248489599531136
- added link Link1, mass 1; collision box size=0.670964103028439 0.9855711403267702 0.7403895370618079; visual box size=0.670964103028439 0.9855711403267702 0.7403895370618079
- added link Link2, mass 1; collision box size=0.400406874452943 0.8993282995531591 0.5150404755113998; visual box size=0.400406874452943 0.8993282995531591 0.5150404755113998
- added link Link3, mass 1; collision box size=0.274795867554725 0.574346255659248 0.7486768818241971; visual box size=0.274795867554725 0.574346255659248 0.7486768818241971
- added link Link4, mass 1; collision box size=0.6031470873200024 0.2620718360123971 0.5157281307400388; visual box size=0.6031470873200024 0.2620718360123971 0.5157281307400388
- added link Link5, mass 1; collision box size=0.2523182819848835 0.2378044836313513 0.20832628410122833; visual box size=0.2523182819848835 0.2378044836313513 0.20832628410122833
- added link Link6, mass 1; collision box size=0.6232050219815071 0.8711560966040075 0.5746742069749482; visual box size=0.6232050219815071 0.8711560966040075 0.5746742069749482
- added link Link7, mass 1; collision box size=0.7232209143649992 0.4651677720300071 0.9109485962113919; visual box size=0.7232209143649992 0.4651677720300071 0.9109485962113919
Joints:
- removed joint BackLeg_LowerBackLeg
- removed joint FrontLeg_LowerFrontLeg
- removed joint LeftLeg_LowerLeftLeg
- removed joint RightLeg_LowerRightLeg
- removed joint Torso_BackLeg
- removed joint Torso_FrontLeg
- removed joint Torso_LeftLeg
- removed joint Torso_RightLeg
- added joint Link0_Link1: type revolute, parent Link0, child Link1, origin xyz=0.3471502316149707 0 0.4624244799765568 rpy=0 0 0, axis 0 1 0, limit lower=-3.14159 upper=3.14159 effort=0.0 velocity=0.0
- added joint Link1_Link2: type revolute, parent Link1, child Link2, origin xyz=0.670964103028439 0 0 rpy=0 0 0, axis 0 1 0, limit lower=-3.14159 upper=3.14159 effort=0.0 velocity=0.0
- added joint Link2_Link3: type revolute, parent Link2, child Link3, origin xyz=0.400406874452943 0 0 rpy=0 0 0, axis 0 1 0, limit lower=-3.14159 upper=3.14159 effort=0.0 velocity=0.0
- added joint Link3_Link4: type revolute, parent Link3, child Link4, origin xyz=0.274795867554725 0 0 rpy=0 0 0, axis 0 1 0, limit lower=-3.14159 upper=3.14159 effort=0.0 velocity=0.0
- added joint Link4_Link5: type revolute, parent Link4, child Link5, origin xyz=0.6031470873200024 0 0 rpy=0 0 0, axis 0 1 0, limit lower=-3.14159 upper=3.14159 effort=0.0 velocity=0.0
- added joint Link5_Link6: type revolute, parent Link5, child Link6, origin xyz=0.2523182819848835 0 0 rpy=0 0 0, axis 0 1 0, limit lower=-3.14159 upper=3.14159 effort=0.0 velocity=0.0
- added joint Link6_Link7: type revolute, parent Link6, child Link7, origin xyz=0.6232050219815071 0 0 rpy=0 0 0, axis 0 1 0, limit lower=-3.14159 upper=3.14159 effort=0.0 velocity=0.0

Commit message: moving snake

File: body.urdf (robot description, URDF)
Before this commit: robot robot, 8 links, 7 joints
Links:
- removed link Link7
- link Link0: geometry collision box size=0.4002836462097963 0.3301060847591615 0.6298899491444221; visual box size=0.4002836462097963 0.3301060847591615 0.6298899491444221
- link Link1: geometry collision box size=0.2274528230275207 0.7742990335961326 0.45970778150162217; visual box size=0.2274528230275207 0.7742990335961326 0.45970778150162217
- link Link2: geometry collision box size=0.3736361300263285 0.5648912231733998 0.20426620335103518; visual box size=0.3736361300263285 0.5648912231733998 0.20426620335103518
- link Link3: geometry collision box size=0.44513834736189434 0.27689229875233407 0.5230120254917963; visual box size=0.44513834736189434 0.27689229875233407 0.5230120254917963
- link Link4: geometry collision box size=0.25001470348057464 0.5618810956089568 0.6324219190053305; visual box size=0.25001470348057464 0.5618810956089568 0.6324219190053305
- link Link5: geometry collision box size=0.6430105298547575 0.20706461278677113 0.69161616662914; visual box size=0.6430105298547575 0.20706461278677113 0.69161616662914
- link Link6: geometry collision box size=0.2182318490915842 0.8044356744781773 0.955765356669765; visual box size=0.2182318490915842 0.8044356744781773 0.955765356669765
Joints:
- removed joint Link6_Link7
- joint Link0_Link1: origin xyz=0.3471502316149707 0 0.4624244799765568 rpy=0 0 0 -> xyz=0.20014182310489814 0 0.31494497457221104 rpy=0 0 0
- joint Link1_Link2: origin xyz=0.670964103028439 0 0 rpy=0 0 0 -> xyz=0.2274528230275207 0 0 rpy=0 0 0
- joint Link2_Link3: origin xyz=0.400406874452943 0 0 rpy=0 0 0 -> xyz=0.3736361300263285 0 0 rpy=0 0 0
- joint Link3_Link4: origin xyz=0.274795867554725 0 0 rpy=0 0 0 -> xyz=0.44513834736189434 0 0 rpy=0 0 0
- joint Link4_Link5: origin xyz=0.6031470873200024 0 0 rpy=0 0 0 -> xyz=0.25001470348057464 0 0 rpy=0 0 0
- joint Link5_Link6: origin xyz=0.2523182819848835 0 0 rpy=0 0 0 -> xyz=0.6430105298547575 0 0 rpy=0 0 0

Commit message: different link colors

File: body.urdf (robot description, URDF)
Before this commit: robot robot, 7 links, 6 joints
Links:
- removed link Link4
- removed link Link5
- removed link Link6
- link Link0: geometry collision box size=0.6952976381060665 0.9307600799723499 0.21643899117873808; visual box size=0.6952976381060665 0.9307600799723499 0.21643899117873808
- link Link1: geometry collision box size=0.9536761504136722 0.6632773543841979 0.9286942433707162; visual box size=0.9536761504136722 0.6632773543841979 0.9286942433707162
- link Link2: geometry collision box size=0.5812286686261479 0.5615816518247922 0.5073541349668629; visual box size=0.5812286686261479 0.5615816518247922 0.5073541349668629
- link Link3: geometry collision box size=0.6351074406693644 0.9005909813643211 0.40837715427933485; visual box size=0.6351074406693644 0.9005909813643211 0.40837715427933485
Joints:
- removed joint Link3_Link4
- removed joint Link4_Link5
- removed joint Link5_Link6
- joint Link0_Link1: origin xyz=0.20014182310489814 0 0.31494497457221104 rpy=0 0 0 -> xyz=0.34764881905303324 0 0.10821949558936904 rpy=0 0 0
- joint Link1_Link2: origin xyz=0.2274528230275207 0 0 rpy=0 0 0 -> xyz=0.9536761504136722 0 0 rpy=0 0 0
- joint Link2_Link3: origin xyz=0.3736361300263285 0 0 rpy=0 0 0 -> xyz=0.5812286686261479 0 0 rpy=0 0 0

Commit message: buggy code for body

File: body.urdf (robot description, URDF)
Before this commit: robot robot, 4 links, 3 joints
Links:
- link Link0: geometry collision box size=0.8655152634319614 0.4934752167574463 0.3764211083016856; visual box size=0.8655152634319614 0.4934752167574463 0.3764211083016856
- link Link1: geometry collision box size=0.5021129420346104 0.20942972424406925 0.7399520471896353; visual box size=0.5021129420346104 0.20942972424406925 0.7399520471896353
- link Link2: geometry collision box size=0.7964525928564536 0.6243921183072609 0.360104944984104; visual box size=0.7964525928564536 0.6243921183072609 0.360104944984104
- link Link3: geometry collision box size=0.7185749712449221 0.6338957164835428 0.5941625252455158; visual box size=0.7185749712449221 0.6338957164835428 0.5941625252455158
Joints:
- joint Link0_Link1: axis 0 1 0 -> 0 0 1; origin xyz=0.34764881905303324 0 0.10821949558936904 rpy=0 0 0 -> xyz=-0.4327576317159807 0 0.1882105541508428 rpy=0 0 0
- joint Link1_Link2: origin xyz=0.9536761504136722 0 0 rpy=0 0 0 -> xyz=0 0 0.5581865777456605 rpy=0 0 0
- joint Link2_Link3: origin xyz=0.5812286686261479 0 0 rpy=0 0 0 -> xyz=0 0 0.008158081658790811 rpy=0 0 0

Commit message: debugging

File: body.urdf (robot description, URDF)
Before this commit: robot robot, 4 links, 3 joints
Links:
- added link Link4, mass 1; collision box size=0.6176003969758552 0.8813163121085004 0.22327659292780766; visual box size=0.6176003969758552 0.8813163121085004 0.22327659292780766
- added link Link5, mass 1; collision box size=0.8602922449469061 0.7769391105850725 0.5969099863964461; visual box size=0.8602922449469061 0.7769391105850725 0.5969099863964461
- added link Link6, mass 1; collision box size=0.9460839855336756 0.21830854024117086 0.3205944171412376; visual box size=0.9460839855336756 0.21830854024117086 0.3205944171412376
- added link Link7, mass 1; collision box size=0.8331662212309554 0.5676324606344787 0.22472281702099936; visual box size=0.8331662212309554 0.5676324606344787 0.22472281702099936
- link Link0: geometry collision box size=0.2196219484783744 0.231167564361364 0.21567420290517916; visual box size=0.2196219484783744 0.231167564361364 0.21567420290517916
- link Link1: geometry collision box size=0.6359975059562332 0.21071331041352598 0.4178001850683688; visual box size=0.6359975059562332 0.21071331041352598 0.4178001850683688
- link Link2: geometry collision box size=0.4721863130982101 0.7496227463509675 0.9749349979497208; visual box size=0.4721863130982101 0.7496227463509675 0.9749349979497208
- link Link3: geometry collision box size=0.33248597160767296 0.44723235013561036 0.9994006107894358; visual box size=0.33248597160767296 0.44723235013561036 0.9994006107894358
Joints:
- added joint Link3_Link4: type revolute, parent Link3, child Link4, origin xyz=0 0.7496227463509675 0 rpy=0 0 0, axis 0 1 0, limit lower=-3.14159 upper=3.14159 effort=0.0 velocity=0.0
- added joint Link4_Link5: type revolute, parent Link4, child Link5, origin xyz=-0.16624298580383648 0.22361617506780518 0 rpy=0 0 0, axis 0 0 1, limit lower=-3.14159 upper=3.14159 effort=0.0 velocity=0.0
- added joint Link5_Link6: type revolute, parent Link5, child Link6, origin xyz=0.23609315654910504 0.37481137317548374 0 rpy=0 0 0, axis 0 1 0, limit lower=-3.14159 upper=3.14159 effort=0.0 velocity=0.0
- added joint Link6_Link7: type revolute, parent Link6, child Link7, origin xyz=-0.4301461224734531 0 0.29845499319822305 rpy=0 0 0, axis 0 1 0, limit lower=-3.14159 upper=3.14159 effort=0.0 velocity=0.0
- joint Link0_Link1: axis 0 0 1 -> 0 1 0; origin xyz=-0.4327576317159807 0 0.1882105541508428 rpy=0 0 0 -> xyz=0 0 0.0 rpy=0 0 0
- joint Link1_Link2: axis 0 1 0 -> 0 0 1; origin xyz=0 0 0.5581865777456605 rpy=0 0 0 -> xyz=0 0.10535665520676299 -0.2089000925341844 rpy=0 0 0
- joint Link2_Link3: origin xyz=0 0 0.008158081658790811 rpy=0 0 0 -> xyz=0 0.115583782180682 0.10783710145258958 rpy=0 0 0

Commit message: debugging

File: body.urdf (robot description, URDF)
Before this commit: robot robot, 8 links, 7 joints
Links:
- removed link Link4
- removed link Link5
- removed link Link6
- removed link Link7
- link Link0: geometry collision box size=0.8505123012958526 0.9064058533970771 0.585377040555846; visual box size=0.8505123012958526 0.9064058533970771 0.585377040555846
- link Link1: geometry collision box size=0.5559544996117177 0.5059242122965839 0.5310858585536806; visual box size=0.5559544996117177 0.5059242122965839 0.5310858585536806
- link Link2: geometry collision box size=0.31838061528661304 0.24878027143768408 0.6654663249975838; visual box size=0.31838061528661304 0.24878027143768408 0.6654663249975838
- link Link3: geometry collision box size=0.2935510992339541 0.21283983434692832 0.494955299636225; visual box size=0.2935510992339541 0.21283983434692832 0.494955299636225
Joints:
- removed joint Link3_Link4
- removed joint Link4_Link5
- removed joint Link5_Link6
- removed joint Link6_Link7
- joint Link0_Link1: origin xyz=0 0 0.0 rpy=0 0 0 -> xyz=0 0.45320292669853857 0.292688520277923 rpy=0 0 0
- joint Link1_Link2: axis 0 0 1 -> 0 1 0; origin xyz=0 0.10535665520676299 -0.2089000925341844 rpy=0 0 0 -> xyz=0.4252561506479263 0 0.292688520277923 rpy=0 0 0
- joint Link2_Link3: origin xyz=0 0.115583782180682 0.10783710145258958 rpy=0 0 0 -> xyz=0 0.25296210614829195 -0.2655429292768403 rpy=0 0 0

Commit message: working

File: body.urdf (robot description, URDF)
Before this commit: robot robot, 4 links, 3 joints
Links:
- link Link0: geometry collision box size=0.2062070453535367 0.7521817507502693 0.2324858468233728; visual box size=0.2062070453535367 0.7521817507502693 0.2324858468233728
- link Link1: geometry collision box size=0.5215656718406843 0.49835438161541906 0.27754836537878386; visual box size=0.5215656718406843 0.49835438161541906 0.27754836537878386
- link Link2: geometry collision box size=0.210189371820937 0.6539872378038349 0.9953226675055649; visual box size=0.210189371820937 0.6539872378038349 0.9953226675055649
- link Link3: geometry collision box size=0.3224524956794532 0.9723688244608601 0.9660231297444144; visual box size=0.3224524956794532 0.9723688244608601 0.9660231297444144
Joints:
- joint Link0_Link1: axis 0 1 0 -> 0 0 1; origin xyz=0 0.45320292669853857 0.292688520277923 rpy=0 0 0 -> xyz=0 0 0.2324858468233728 rpy=0 0 0
- joint Link1_Link2: origin xyz=0.4252561506479263 0 0.292688520277923 rpy=0 0 0 -> xyz=0 0 0.2324858468233728 rpy=0 0 0
- joint Link2_Link3: origin xyz=0 0.25296210614829195 -0.2655429292768403 rpy=0 0 0 -> xyz=-0.2607828359203421 0 0.13877418268939193 rpy=0 0 0

Commit message: debugging

File: body.urdf (robot description, URDF)
Before this commit: robot robot, 4 links, 3 joints
Links:
- added link Link4, mass 1; collision box size=-1.3877787807814457e-17 -0.2891350604314722 0.5282970053497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; visual box size=-1.3877787807814457e-17 -0.2891350604314722 0.5282970053497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
- added link Link5, mass 1; collision box size=0.0 -0.47385262549896795 -0.2068995510378766; visual box size=0.0 -0.47385262549896795 -0.2068995510378766
- link Link0: geometry collision box size=0.2511004352223453 0.5778564897835979 0.9159456502421126; visual box size=0.2511004352223453 0.5778564897835979 0.9159456502421126
- link Link1: geometry collision box size=-0.016551482953381685 0.7534289407085111 0.8937406564076413; visual box size=-0.016551482953381685 0.7534289407085111 0.8937406564076413
- link Link2: geometry collision box size=0.0 0.32456196590615183 0.5120955077454246; visual box size=0.0 0.32456196590615183 0.5120955077454246
- link Link3: geometry collision box size=-2.7755575615628914e-17 -1.1074791572866882 0.5220395327191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; visual box size=-2.7755575615628914e-17 -1.1074791572866882 0.5220395327191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
Joints:
- added joint Link3_Link4: type revolute, parent Link3, child Link4, origin xyz=0 0 0.8937406564076413 rpy=0 0 0, axis 1 0 0, limit lower=-3.14159 upper=3.14159 effort=0.0 velocity=0.0
- added joint Link4_Link5: type revolute, parent Link4, child Link5, origin xyz=0 -0.1445675302157361 0.2641485026748935 rpy=0 0 0, axis 1 0 0, limit lower=-3.14159 upper=3.14159 effort=0.0 velocity=0.0
- joint Link0_Link1: origin xyz=0 0 0.2324858468233728 rpy=0 0 0 -> xyz=0 0 0.9159456502421126 rpy=0 0 0
- joint Link1_Link2: axis 0 1 0 -> 0 0 1; origin xyz=0 0 0.2324858468233728 rpy=0 0 0 -> xyz=0 0.37671447035425554 0.44687032820382067 rpy=0 0 0
- joint Link2_Link3: axis 0 1 0 -> 0 0 1; origin xyz=-0.2607828359203421 0 0.13877418268939193 rpy=0 0 0 -> xyz=0 -0.28892824489179897 0.4579728251210563 rpy=0 0 0

Commit message: kinda works

File: body.urdf (robot description, URDF)
Before this commit: robot robot, 6 links, 5 joints
Links:
- link Link0: geometry collision box size=0.38674226633997916 0.7664143733226927 0.5732765423310966; visual box size=0.38674226633997916 0.7664143733226927 0.5732765423310966
- link Link1: geometry collision box size=0.7660168086497421 0.6634770824077074 0.3651340563480505; visual box size=0.7660168086497421 0.6634770824077074 0.3651340563480505
- link Link2: geometry collision box size=0.699733065428906 0.5692244338311904 0.34308016822587006; visual box size=0.699733065428906 0.5692244338311904 0.34308016822587006
- link Link3: geometry collision box size=0.3752835279839607 0.9436974682904191 0.23587325766859585; visual box size=0.3752835279839607 0.9436974682904191 0.23587325766859585
- link Link4: geometry collision box size=0.9978591745973122 0.21236120844264478 0.2926294197746446; visual box size=0.9978591745973122 0.21236120844264478 0.2926294197746446
- link Link5: geometry collision box size=0.5911359032932514 0.7291191467932967 0.45996746921929677; visual box size=0.5911359032932514 0.7291191467932967 0.45996746921929677
Joints:
- joint Link0_Link1: axis 0 0 1 -> 1 0 0; origin xyz=0 0 0.9159456502421126 rpy=0 0 0 -> xyz=0 -0.38320718666134634 0.2866382711655483 rpy=0 0 0
- joint Link1_Link2: axis 0 0 1 -> 1 0 0; origin xyz=0 0.37671447035425554 0.44687032820382067 rpy=0 0 0 -> xyz=0 -0.3317385412038537 0.18256702817402526 rpy=0 0 0
- joint Link2_Link3: axis 0 0 1 -> 0 1 0; origin xyz=0 -0.28892824489179897 0.4579728251210563 rpy=0 0 0 -> xyz=-0.38300840432487104 -0.3317385412038537 0 rpy=0 0 0
- joint Link3_Link4: axis 1 0 0 -> 0 1 0; origin xyz=0 0 0.8937406564076413 rpy=0 0 0 -> xyz=0.19337113316998958 0 0.2866382711655483 rpy=0 0 0
- joint Link4_Link5: origin xyz=0 -0.1445675302157361 0.2641485026748935 rpy=0 0 0 -> xyz=0.4989295872986561 -0.10618060422132239 0 rpy=0 0 0

Commit message: debug

File: body.urdf (robot description, URDF)
Before this commit: robot robot, 6 links, 5 joints
Links:
- removed link Link3
- removed link Link4
- removed link Link5
- link Link0: geometry collision box size=0.2263642155711163 0.8971948235423992 0.22775841589471402; visual box size=0.2263642155711163 0.8971948235423992 0.22775841589471402
- link Link1: geometry collision box size=0.5048012297630615 0.546072060279839 0.6069374575109735; visual box size=0.5048012297630615 0.546072060279839 0.6069374575109735
- link Link2: geometry collision box size=0.4731694490260573 0.3594095536677611 0.561037156971885; visual box size=0.4731694490260573 0.3594095536677611 0.561037156971885
Joints:
- removed joint Link2_Link3
- removed joint Link3_Link4
- removed joint Link4_Link5
- joint Link0_Link1: axis 1 0 0 -> 0 1 0; origin xyz=0 -0.38320718666134634 0.2866382711655483 rpy=0 0 0 -> xyz=0 0.4485974117711996 0.11387920794735701 rpy=0 0 0
- joint Link1_Link2: axis 1 0 0 -> 0 0 1; origin xyz=0 -0.3317385412038537 0.18256702817402526 rpy=0 0 0 -> xyz=0.5048012297630615 0 0 rpy=0 0 0

Commit message: Revert "debug"
This reverts commit 9a1687e1cfd6b8317faa7cb8ea66c25c57a1dc35.

did something wrong

File: body.urdf (robot description, URDF)
Before this commit: robot robot, 3 links, 2 joints
Links:
- added link Link3, mass 1; collision box size=0.3752835279839607 0.9436974682904191 0.23587325766859585; visual box size=0.3752835279839607 0.9436974682904191 0.23587325766859585
- added link Link4, mass 1; collision box size=0.9978591745973122 0.21236120844264478 0.2926294197746446; visual box size=0.9978591745973122 0.21236120844264478 0.2926294197746446
- added link Link5, mass 1; collision box size=0.5911359032932514 0.7291191467932967 0.45996746921929677; visual box size=0.5911359032932514 0.7291191467932967 0.45996746921929677
- link Link0: geometry collision box size=0.38674226633997916 0.7664143733226927 0.5732765423310966; visual box size=0.38674226633997916 0.7664143733226927 0.5732765423310966
- link Link1: geometry collision box size=0.7660168086497421 0.6634770824077074 0.3651340563480505; visual box size=0.7660168086497421 0.6634770824077074 0.3651340563480505
- link Link2: geometry collision box size=0.699733065428906 0.5692244338311904 0.34308016822587006; visual box size=0.699733065428906 0.5692244338311904 0.34308016822587006
Joints:
- added joint Link2_Link3: type revolute, parent Link2, child Link3, origin xyz=-0.38300840432487104 -0.3317385412038537 0 rpy=0 0 0, axis 0 1 0, limit lower=-3.14159 upper=3.14159 effort=0.0 velocity=0.0
- added joint Link3_Link4: type revolute, parent Link3, child Link4, origin xyz=0.19337113316998958 0 0.2866382711655483 rpy=0 0 0, axis 0 1 0, limit lower=-3.14159 upper=3.14159 effort=0.0 velocity=0.0
- added joint Link4_Link5: type revolute, parent Link4, child Link5, origin xyz=0.4989295872986561 -0.10618060422132239 0 rpy=0 0 0, axis 1 0 0, limit lower=-3.14159 upper=3.14159 effort=0.0 velocity=0.0
- joint Link0_Link1: axis 0 1 0 -> 1 0 0; origin xyz=0 0.4485974117711996 0.11387920794735701 rpy=0 0 0 -> xyz=0 -0.38320718666134634 0.2866382711655483 rpy=0 0 0
- joint Link1_Link2: axis 0 0 1 -> 1 0 0; origin xyz=0.5048012297630615 0 0 rpy=0 0 0 -> xyz=0 -0.3317385412038537 0.18256702817402526 rpy=0 0 0
