Commit message: fixed joint positions

File: body.urdf (robot description, URDF)
Before this commit: robot robot, 6 links, 5 joints
Links:
- link Link0: geometry collision box size=0.8962544266781778 0.9305835131628204 0.9482579050850259; visual box size=0.8962544266781778 0.9305835131628204 0.9482579050850259
- link Link1: geometry collision box size=0.5159493384318312 0.6288551071809552 0.973747269710366; visual box size=0.5159493384318312 0.6288551071809552 0.973747269710366
- link Link2: geometry collision box size=0.8238933405985807 0.9125890881022025 0.3229275272559856; visual box size=0.8238933405985807 0.9125890881022025 0.3229275272559856
- link Link3: geometry collision box size=0.2832035550972955 0.8983869001768545 0.9421578035489351; visual box size=0.2832035550972955 0.8983869001768545 0.9421578035489351
- link Link4: geometry collision box size=0.7337882999578238 0.7691769721112736 0.8606301076345833; visual box size=0.7337882999578238 0.7691769721112736 0.8606301076345833
- link Link5: geometry collision box size=0.29669123636509975 0.5173055238260309 0.732514419335913; visual box size=0.29669123636509975 0.5173055238260309 0.732514419335913
Joints:
- removed joint Link1_Link2
- removed joint Link2_Link3
- removed joint Link3_Link4
- added joint Link0_Link2: type revolute, parent Link0, child Link2, origin xyz=0 0 0.9482579050850259 rpy=0 0 0, axis 0 1 0, limit lower=-3.14159 upper=3.14159 effort=0.0 velocity=0.0
- added joint Link0_Link4: type revolute, parent Link0, child Link4, origin xyz=0 0.4652917565814102 0.47412895254251297 rpy=0 0 0, axis 0 1 0, limit lower=-3.14159 upper=3.14159 effort=0.0 velocity=0.0
- added joint Link1_Link3: type revolute, parent Link1, child Link3, origin xyz=0 -0.3144275535904776 -0.486873634855183 rpy=0 0 0, axis 1 0 0, limit lower=-3.14159 upper=3.14159 effort=0.0 velocity=0.0
- joint Link0_Link1: origin xyz=0 -0.38320718666134634 0.2866382711655483 rpy=0 0 0 -> xyz=0 -0.4652917565814102 0.47412895254251297 rpy=0 0 0
- joint Link4_Link5: axis 1 0 0 -> 0 0 1; origin xyz=0.4989295872986561 -0.10618060422132239 0 rpy=0 0 0 -> xyz=0 0.3845884860556368 0.4303150538172916 rpy=0 0 0
