Commit message: start evolution

File: body0.urdf (robot description, URDF)
Before this commit: robot robot, 4 links, 3 joints
Links:
- link Link0: geometry collision box size=0.22863825967406523 0.7530109358968506 0.705035803511026; visual box size=0.22863825967406523 0.7530109358968506 0.705035803511026
- link Link1: geometry collision box size=0.2934158928506494 0.4850722630682553 0.32011126655920963; visual box size=0.2934158928506494 0.4850722630682553 0.32011126655920963
- link Link2: geometry collision box size=0.9506507987540478 0.42695957597998285 0.4436722870067213; visual box size=0.9506507987540478 0.42695957597998285 0.4436722870067213
- link Link3: geometry collision box size=0.2884187637373506 0.7445226902121356 0.4230736496275775; visual box size=0.2884187637373506 0.7445226902121356 0.4230736496275775
Joints:
- removed joint Link1_Link2
- removed joint Link1_Link3
- added joint Link0_Link2: type revolute, parent Link0, child Link2, origin xyz=0.11431912983703262 0 0.352517901755513 rpy=0 0 0, axis 0 1 0, limit lower=-3.14159 upper=3.14159 effort=0.0 velocity=0.0
- added joint Link2_Link3: type revolute, parent Link2, child Link3, origin xyz=0.9506507987540478 0 0 rpy=0 0 0, axis 0 1 0, limit lower=-3.14159 upper=3.14159 effort=0.0 velocity=0.0
- joint Link0_Link1: origin xyz=0 0 0.6544720429988153 rpy=0 0 0 -> xyz=0 -0.3765054679484253 0.352517901755513 rpy=0 0 0

File: body12.urdf (robot description, URDF)
Before this commit: robot robot, 4 links, 3 joints
Links:
- link Link0: geometry collision box size=0.8327148101492399 0.25569459198704436 0.5574464453252742; visual box size=0.8327148101492399 0.25569459198704436 0.5574464453252742
- link Link1: geometry collision box size=0.22360662325441735 0.9826698895665642 0.6394693361375642; visual box size=0.22360662325441735 0.9826698895665642 0.6394693361375642
- link Link2: geometry collision box size=0.7324933614011544 0.997944552355621 0.2225377053767253; visual box size=0.7324933614011544 0.997944552355621 0.2225377053767253
- link Link3: geometry collision box size=0.5265573049184509 0.63752336921159 0.43975406686129076; visual box size=0.5265573049184509 0.63752336921159 0.43975406686129076
Joints:
- joint Link0_Link1: axis 0 0 1 -> 0 1 0; origin xyz=0 0 0.6544720429988153 rpy=0 0 0 -> xyz=0 0 0.5574464453252742 rpy=0 0 0
- joint Link1_Link2: axis 0 1 0 -> 0 0 1; origin xyz=0.3666074044375889 0 0.35143184973512376 rpy=0 0 0 -> xyz=0 0.4913349447832821 0.3197346680687821 rpy=0 0 0
- joint Link1_Link3: axis 1 0 0 -> 0 0 1; origin xyz=0 0.3693474804029421 0.35143184973512376 rpy=0 0 0 -> xyz=0 0 0.6394693361375642 rpy=0 0 0

File: body15.urdf (robot description, URDF)
Before this commit: robot robot, 4 links, 3 joints
Links:
- link Link0: geometry collision box size=0.28761541259314777 0.34689391757525795 0.7212157681057936; visual box size=0.28761541259314777 0.34689391757525795 0.7212157681057936
- link Link1: geometry collision box size=0.9282163704206605 0.644510746496533 0.2052427523692905; visual box size=0.9282163704206605 0.644510746496533 0.2052427523692905
- link Link2: geometry collision box size=0.4819456225815204 0.426275613587672 0.8101253005127822; visual box size=0.4819456225815204 0.426275613587672 0.8101253005127822
- link Link3: geometry collision box size=0.8252386890419501 0.5675809817075852 0.9358506333638077; visual box size=0.8252386890419501 0.5675809817075852 0.9358506333638077
Joints:
- removed joint Link1_Link2
- removed joint Link1_Link3
- added joint Link0_Link2: type revolute, parent Link0, child Link2, origin xyz=-0.14380770629657388 0 0.3606078840528968 rpy=0 0 0, axis 0 0 1, limit lower=-3.14159 upper=3.14159 effort=0.0 velocity=0.0
- added joint Link2_Link3: type revolute, parent Link2, child Link3, origin xyz=-0.2409728112907602 0.213137806793836 0 rpy=0 0 0, axis 1 0 0, limit lower=-3.14159 upper=3.14159 effort=0.0 velocity=0.0
- joint Link0_Link1: origin xyz=0 0 0.6544720429988153 rpy=0 0 0 -> xyz=0 0 0.7212157681057936 rpy=0 0 0

File: body18.urdf (robot description, URDF)
Before this commit: robot robot, 4 links, 3 joints
Links:
- link Link0: geometry collision box size=0.6787613042713205 0.8419545116554628 0.22967159658332223; visual box size=0.6787613042713205 0.8419545116554628 0.22967159658332223
- link Link1: geometry collision box size=0.962670224805966 0.2163240907823754 0.6113734922886955; visual box size=0.962670224805966 0.2163240907823754 0.6113734922886955
- link Link2: geometry collision box size=0.21544117221213357 0.5474208366786013 0.5638861262888824; visual box size=0.21544117221213357 0.5474208366786013 0.5638861262888824
- link Link3: geometry collision box size=0.6118065905779686 0.9357109318446313 0.8064981708686485; visual box size=0.6118065905779686 0.9357109318446313 0.8064981708686485
Joints:
- removed joint Link1_Link3
- added joint Link2_Link3: type revolute, parent Link2, child Link3, origin xyz=0 0 0.5638861262888824 rpy=0 0 0, axis 0 1 0, limit lower=-3.14159 upper=3.14159 effort=0.0 velocity=0.0
- joint Link0_Link1: origin xyz=0 0 0.6544720429988153 rpy=0 0 0 -> xyz=0.33938065213566027 0 0.11483579829166111 rpy=0 0 0
- joint Link1_Link2: axis 0 1 0 -> 1 0 0; origin xyz=0.3666074044375889 0 0.35143184973512376 rpy=0 0 0 -> xyz=0.481335112402983 0 0.30568674614434777 rpy=0 0 0

File: body21.urdf (robot description, URDF)
Before this commit: robot robot, 4 links, 3 joints
Links:
- link Link0: geometry collision box size=0.8619626580188189 0.8807647254636184 0.6167424199231446; visual box size=0.8619626580188189 0.8807647254636184 0.6167424199231446
- link Link1: geometry collision box size=0.7240723293094806 0.5932149526681407 0.952265398490115; visual box size=0.7240723293094806 0.5932149526681407 0.952265398490115
- link Link2: geometry collision box size=0.24192112226870668 0.6916639051070563 0.8400137816716671; visual box size=0.24192112226870668 0.6916639051070563 0.8400137816716671
- link Link3: geometry collision box size=0.28218518426672157 0.5120920278934659 0.6388777578651813; visual box size=0.28218518426672157 0.5120920278934659 0.6388777578651813
Joints:
- removed joint Link1_Link2
- removed joint Link1_Link3
- added joint Link0_Link2: type revolute, parent Link0, child Link2, origin xyz=0 -0.4403823627318092 0.3083712099615723 rpy=0 0 0, axis 1 0 0, limit lower=-3.14159 upper=3.14159 effort=0.0 velocity=0.0
- added joint Link2_Link3: type revolute, parent Link2, child Link3, origin xyz=-0.12096056113435334 -0.34583195255352817 0 rpy=0 0 0, axis 1 0 0, limit lower=-3.14159 upper=3.14159 effort=0.0 velocity=0.0
- joint Link0_Link1: axis 0 0 1 -> 1 0 0; origin xyz=0 0 0.6544720429988153 rpy=0 0 0 -> xyz=0 0 0.6167424199231446 rpy=0 0 0

File: body24.urdf (robot description, URDF)
Before this commit: robot robot, 4 links, 3 joints
Links:
- link Link0: geometry collision box size=0.3749932258556287 0.9719343053719138 0.2933653718626862; visual box size=0.3749932258556287 0.9719343053719138 0.2933653718626862
- link Link1: geometry collision box size=0.6768489643570265 0.221692051023921 0.7359321481271; visual box size=0.6768489643570265 0.221692051023921 0.7359321481271
- link Link2: geometry collision box size=0.9042485346502596 0.5609612428195192 0.6715538801749612; visual box size=0.9042485346502596 0.5609612428195192 0.6715538801749612
- link Link3: geometry collision box size=0.36844020336761274 0.9468994848824444 0.7888473154811155; visual box size=0.36844020336761274 0.9468994848824444 0.7888473154811155
Joints:
- removed joint Link1_Link3
- added joint Link2_Link3: type revolute, parent Link2, child Link3, origin xyz=0 0.2804806214097596 -0.3357769400874806 rpy=0 0 0, axis 0 0 1, limit lower=-3.14159 upper=3.14159 effort=0.0 velocity=0.0
- joint Link0_Link1: axis 0 0 1 -> 1 0 0; origin xyz=0 0 0.6544720429988153 rpy=0 0 0 -> xyz=0 0.4859671526859569 0.1466826859313431 rpy=0 0 0
- joint Link1_Link2: axis 0 1 0 -> 0 0 1; origin xyz=0.3666074044375889 0 0.35143184973512376 rpy=0 0 0 -> xyz=0 0.1108460255119605 -0.36796607406355 rpy=0 0 0

File: body27.urdf (robot description, URDF)
Before this commit: robot robot, 4 links, 3 joints
Links:
- link Link0: geometry collision box size=0.28767792420679283 0.48300308116214813 0.309978453498154; visual box size=0.28767792420679283 0.48300308116214813 0.309978453498154
- link Link1: geometry collision box size=0.539517620244766 0.7934985037697724 0.3612163537631342; visual box size=0.539517620244766 0.7934985037697724 0.3612163537631342
- link Link2: geometry collision box size=0.6683415262614246 0.3261753732573907 0.7653338810400798; visual box size=0.6683415262614246 0.3261753732573907 0.7653338810400798
- link Link3: geometry collision box size=0.6962704987910147 0.25249663773407516 0.4983444516891165; visual box size=0.6962704987910147 0.25249663773407516 0.4983444516891165
Joints:
- removed joint Link1_Link2
- removed joint Link1_Link3
- added joint Link0_Link2: type revolute, parent Link0, child Link2, origin xyz=0 -0.24150154058107406 0.154989226749077 rpy=0 0 0, axis 1 0 0, limit lower=-3.14159 upper=3.14159 effort=0.0 velocity=0.0
- added joint Link2_Link3: type revolute, parent Link2, child Link3, origin xyz=0 -0.16308768662869536 0.3826669405200399 rpy=0 0 0, axis 0 0 1, limit lower=-3.14159 upper=3.14159 effort=0.0 velocity=0.0
- joint Link0_Link1: origin xyz=0 0 0.6544720429988153 rpy=0 0 0 -> xyz=0 0.24150154058107406 0.154989226749077 rpy=0 0 0

File: body3.urdf (robot description, URDF)
Before this commit: robot robot, 4 links, 3 joints
Links:
- link Link0: geometry collision box size=0.7893771966329843 0.3893841688204444 0.26922055874636197; visual box size=0.7893771966329843 0.3893841688204444 0.26922055874636197
- link Link1: geometry collision box size=0.518984669173826 0.7054757924969606 0.2772789773644956; visual box size=0.518984669173826 0.7054757924969606 0.2772789773644956
- link Link2: geometry collision box size=0.3582414358469129 0.46504911933690485 0.7551768557973488; visual box size=0.3582414358469129 0.46504911933690485 0.7551768557973488
- link Link3: geometry collision box size=0.824726926475871 0.9353321259741749 0.9607644749474564; visual box size=0.824726926475871 0.9353321259741749 0.9607644749474564
Joints:
- joint Link0_Link1: axis 0 0 1 -> 1 0 0; origin xyz=0 0 0.6544720429988153 rpy=0 0 0 -> xyz=0 0.1946920844102222 0.13461027937318099 rpy=0 0 0
- joint Link1_Link2: origin xyz=0.3666074044375889 0 0.35143184973512376 rpy=0 0 0 -> xyz=0.259492334586913 0.3527378962484803 0 rpy=0 0 0
- joint Link1_Link3: axis 1 0 0 -> 0 1 0; origin xyz=0 0.3693474804029421 0.35143184973512376 rpy=0 0 0 -> xyz=-0.259492334586913 0.3527378962484803 0 rpy=0 0 0

File: body30.urdf (robot description, URDF)
Before this commit: robot robot, 4 links, 3 joints
Links:
- link Link0: geometry collision box size=0.7366512833284635 0.5678325058203894 0.9821942789059823; visual box size=0.7366512833284635 0.5678325058203894 0.9821942789059823
- link Link1: geometry collision box size=0.2804289834173601 0.2156148029775823 0.820561870822665; visual box size=0.2804289834173601 0.2156148029775823 0.820561870822665
- link Link2: geometry collision box size=0.6873645906128476 0.28494182240469357 0.9959733930863393; visual box size=0.6873645906128476 0.28494182240469357 0.9959733930863393
- link Link3: geometry collision box size=0.7041432913412151 0.5370380803042596 0.2337421115920451; visual box size=0.7041432913412151 0.5370380803042596 0.2337421115920451
Joints:
- removed joint Link1_Link2
- removed joint Link1_Link3
- added joint Link0_Link2: type revolute, parent Link0, child Link2, origin xyz=0 -0.2839162529101947 0.49109713945299116 rpy=0 0 0, axis 0 1 0, limit lower=-3.14159 upper=3.14159 effort=0.0 velocity=0.0
- added joint Link0_Link3: type revolute, parent Link0, child Link3, origin xyz=-0.36832564166423176 0 0.49109713945299116 rpy=0 0 0, axis 1 0 0, limit lower=-3.14159 upper=3.14159 effort=0.0 velocity=0.0
- joint Link0_Link1: axis 0 0 1 -> 1 0 0; origin xyz=0 0 0.6544720429988153 rpy=0 0 0 -> xyz=0 0.2839162529101947 0.49109713945299116 rpy=0 0 0

File: body6.urdf (robot description, URDF)
Before this commit: robot robot, 4 links, 3 joints
Links:
- link Link0: geometry collision box size=0.8347666733602486 0.642417319121094 0.9601396841293193; visual box size=0.8347666733602486 0.642417319121094 0.9601396841293193
- link Link1: geometry collision box size=0.6414583958258888 0.404748717874376 0.8540500100379929; visual box size=0.6414583958258888 0.404748717874376 0.8540500100379929
- link Link2: geometry collision box size=0.7776022794098856 0.9353450061539159 0.8880562290863829; visual box size=0.7776022794098856 0.9353450061539159 0.8880562290863829
- link Link3: geometry collision box size=0.990175535294709 0.7435029115517007 0.2688114712510995; visual box size=0.990175535294709 0.7435029115517007 0.2688114712510995
Joints:
- removed joint Link1_Link2
- added joint Link0_Link2: type revolute, parent Link0, child Link2, origin xyz=0 0 0.9601396841293193 rpy=0 0 0, axis 0 0 1, limit lower=-3.14159 upper=3.14159 effort=0.0 velocity=0.0
- joint Link0_Link1: axis 0 0 1 -> 1 0 0; origin xyz=0 0 0.6544720429988153 rpy=0 0 0 -> xyz=0.4173833366801243 0 0.48006984206465964 rpy=0 0 0
- joint Link1_Link3: axis 1 0 0 -> 0 0 1; origin xyz=0 0.3693474804029421 0.35143184973512376 rpy=0 0 0 -> xyz=0.3207291979129444 0 -0.42702500501899643 rpy=0 0 0

File: body9.urdf (robot description, URDF)
Before this commit: robot robot, 4 links, 3 joints
Links:
- link Link0: geometry collision box size=0.6028039009280342 0.446334971432933 0.384131811178158; visual box size=0.6028039009280342 0.446334971432933 0.384131811178158
- link Link1: geometry collision box size=0.27033237451948255 0.8758065318572927 0.38963279439295606; visual box size=0.27033237451948255 0.8758065318572927 0.38963279439295606
- link Link2: geometry collision box size=0.7370833065965177 0.5075208673234999 0.24942180169718695; visual box size=0.7370833065965177 0.5075208673234999 0.24942180169718695
- link Link3: geometry collision box size=0.7340574458651832 0.24151224025217238 0.45877031747853203; visual box size=0.7340574458651832 0.24151224025217238 0.45877031747853203
Joints:
- removed joint Link1_Link2
- added joint Link0_Link2: type revolute, parent Link0, child Link2, origin xyz=-0.3014019504640171 0 0.192065905589079 rpy=0 0 0, axis 1 0 0, limit lower=-3.14159 upper=3.14159 effort=0.0 velocity=0.0
- joint Link0_Link1: axis 0 0 1 -> 1 0 0; origin xyz=0 0 0.6544720429988153 rpy=0 0 0 -> xyz=0.3014019504640171 0 0.192065905589079 rpy=0 0 0
- joint Link1_Link3: axis 1 0 0 -> 0 1 0; origin xyz=0 0.3693474804029421 0.35143184973512376 rpy=0 0 0 -> xyz=0.13516618725974128 -0.43790326592864637 0 rpy=0 0 0

Commit message: debug

File: body0.urdf (robot description, URDF)
Before this commit: robot robot, 6 links, 5 joints
Links:
- added link Link6, mass 1; collision box size=0.22755149870614133 0.5663424266801047 0.6326850459064899; visual box size=0.22755149870614133 0.5663424266801047 0.6326850459064899
- link Link0: geometry collision box size=0.5007499518699512 0.2478970985959859 0.4279964667106767; visual box size=0.5007499518699512 0.2478970985959859 0.4279964667106767
- link Link1: geometry collision box size=0.27273245394168566 0.8941272285731923 0.5715063274434113; visual box size=0.27273245394168566 0.8941272285731923 0.5715063274434113
- link Link2: geometry collision box size=0.6167083259279713 0.5280727702730748 0.40146910955610465; visual box size=0.6167083259279713 0.5280727702730748 0.40146910955610465
- link Link3: geometry collision box size=0.4652356559635351 0.28208255785454633 0.3979862799923002; visual box size=0.4652356559635351 0.28208255785454633 0.3979862799923002
- link Link4: geometry collision box size=0.3917566297325206 0.9664195937875497 0.2072709624811643; visual box size=0.3917566297325206 0.9664195937875497 0.2072709624811643
- link Link5: geometry collision box size=0.462474650272928 0.9313012052633642 0.2123593357464059; visual box size=0.462474650272928 0.9313012052633642 0.2123593357464059
Joints:
- removed joint Link0_Link2
- removed joint Link2_Link5
- removed joint Link3_Link4
- added joint Link1_Link2: type revolute, parent Link1, child Link2, origin xyz=0 0 0.5715063274434113 rpy=0 0 0, axis 0 0 1, limit lower=-3.14159 upper=3.14159 effort=0.0 velocity=0.0
- added joint Link1_Link5: type revolute, parent Link1, child Link5, origin xyz=0 -0.44706361428659613 0.28575316372170567 rpy=0 0 0, axis 1 0 0, limit lower=-3.14159 upper=3.14159 effort=0.0 velocity=0.0
- added joint Link2_Link4: type revolute, parent Link2, child Link4, origin xyz=0 0.2640363851365374 0.20073455477805233 rpy=0 0 0, axis 0 0 1, limit lower=-3.14159 upper=3.14159 effort=0.0 velocity=0.0
- added joint Link2_Link6: type revolute, parent Link2, child Link6, origin xyz=0 -0.2640363851365374 0.20073455477805233 rpy=0 0 0, axis 0 1 0, limit lower=-3.14159 upper=3.14159 effort=0.0 velocity=0.0
- joint Link0_Link1: axis 1 0 0 -> 0 1 0; origin xyz=0 0 0.5598087793815415 rpy=0 0 0 -> xyz=0 0 0.4279964667106767 rpy=0 0 0
- joint Link2_Link3: axis 0 0 1 -> 1 0 0; origin xyz=0 -0.44920843685609635 0.2568943195408061 rpy=0 0 0 -> xyz=0 0 0.40146910955610465 rpy=0 0 0

File: body1.urdf (robot description, URDF)
Before this commit: robot robot, 6 links, 5 joints
Links:
- added link Link6, mass 1; collision box size=0.3893551058564126 0.5108001592045947 0.9923509871127381; visual box size=0.3893551058564126 0.5108001592045947 0.9923509871127381
- link Link0: geometry collision box size=0.32673917484087434 0.6506584473071308 0.4397788389053114; visual box size=0.32673917484087434 0.6506584473071308 0.4397788389053114
- link Link1: geometry collision box size=0.22454393727644542 0.9984343503332433 0.6359254162011483; visual box size=0.22454393727644542 0.9984343503332433 0.6359254162011483
- link Link2: geometry collision box size=0.2498672422369234 0.20085590293104688 0.6252468129432989; visual box size=0.2498672422369234 0.20085590293104688 0.6252468129432989
- link Link3: geometry collision box size=0.7975051695254591 0.952164521085479 0.29368155220777326; visual box size=0.7975051695254591 0.952164521085479 0.29368155220777326
- link Link4: geometry collision box size=0.2068736308702831 0.7543406670506487 0.8220224439601391; visual box size=0.2068736308702831 0.7543406670506487 0.8220224439601391
- link Link5: geometry collision box size=0.4731394222513512 0.8187207157817415 0.5017332677105286; visual box size=0.4731394222513512 0.8187207157817415 0.5017332677105286
Joints:
- removed joint Link0_Link3
- removed joint Link0_Link4
- added joint Link1_Link3: type revolute, parent Link1, child Link3, origin xyz=0 -0.4992171751666217 0.31796270810057414 rpy=0 0 0, axis 0 0 1, limit lower=-3.14159 upper=3.14159 effort=0.0 velocity=0.0
- added joint Link2_Link4: type revolute, parent Link2, child Link4, origin xyz=0 0.20085590293104688 0 rpy=0 0 0, axis 0 0 1, limit lower=-3.14159 upper=3.14159 effort=0.0 velocity=0.0
- added joint Link3_Link6: type revolute, parent Link3, child Link6, origin xyz=0 -0.4760822605427395 0.14684077610388663 rpy=0 0 0, axis 1 0 0, limit lower=-3.14159 upper=3.14159 effort=0.0 velocity=0.0
- joint Link0_Link1: axis 0 0 1 -> 1 0 0; origin xyz=0 0.46665299900455015 0.4329834080671191 rpy=0 0 0 -> xyz=0 0 0.4397788389053114 rpy=0 0 0
- joint Link1_Link2: axis 0 1 0 -> 0 0 1; origin xyz=0 0.0 0 rpy=0 0 0 -> xyz=0 0.4992171751666217 0.31796270810057414 rpy=0 0 0
- joint Link3_Link5: origin xyz=0 -0.32283597689523164 0 rpy=0 0 0 -> xyz=0 0.0 0 rpy=0 0 0

Commit message: robot moving again

File: body0.urdf (robot description, URDF)
Before this commit: robot robot, 7 links, 6 joints
Links:
- removed link Link5
- removed link Link6
- link Link0: geometry collision box size=0.49222885497054225 0.5725636893709081 0.5772515811924539; visual box size=0.49222885497054225 0.5725636893709081 0.5772515811924539
- link Link1: geometry collision box size=0.26917906905728106 0.3971983633409346 0.6979934727572723; visual box size=0.26917906905728106 0.3971983633409346 0.6979934727572723
- link Link2: geometry collision box size=0.632459074375797 0.7919461307819684 0.5520122301356494; visual box size=0.632459074375797 0.7919461307819684 0.5520122301356494
- link Link3: geometry collision box size=0.5363076517631122 0.7686986689649389 0.22531307360626648; visual box size=0.5363076517631122 0.7686986689649389 0.22531307360626648
- link Link4: geometry collision box size=0.31454991730079823 0.49464848234716446 0.28121889528573096; visual box size=0.31454991730079823 0.49464848234716446 0.28121889528573096
Joints:
- removed joint Link1_Link2
- removed joint Link1_Link5
- removed joint Link2_Link4
- removed joint Link2_Link6
- added joint Link0_Link2: type revolute, parent Link0, child Link2, origin xyz=0 0 0.5772515811924539 rpy=0 0 0, axis 0 1 0, limit lower=-3.14159 upper=3.14159 effort=0.0 velocity=0.0
- added joint Link1_Link4: type revolute, parent Link1, child Link4, origin xyz=0 -0.1985991816704673 0.34899673637863615 rpy=0 0 0, axis 0 0 1, limit lower=-3.14159 upper=3.14159 effort=0.0 velocity=0.0
- joint Link0_Link1: origin xyz=0 0 0.4279964667106767 rpy=0 0 0 -> xyz=0 0 0.5772515811924539 rpy=0 0 0
- joint Link2_Link3: axis 1 0 0 -> 0 1 0; origin xyz=0 0 0.40146910955610465 rpy=0 0 0 -> xyz=0 -0.3959730653909842 0.2760061150678247 rpy=0 0 0

File: body1.urdf (robot description, URDF)
Before this commit: robot robot, 7 links, 6 joints
Links:
- removed link Link5
- removed link Link6
- link Link0: geometry collision box size=0.2812699331641804 0.5802022735954849 0.2227436123548494; visual box size=0.2812699331641804 0.5802022735954849 0.2227436123548494
- link Link1: geometry collision box size=0.7503146365481035 0.8651793722361623 0.9613545967195773; visual box size=0.7503146365481035 0.8651793722361623 0.9613545967195773
- link Link2: geometry collision box size=0.26872934650523495 0.7807701555987012 0.4726564020922365; visual box size=0.26872934650523495 0.7807701555987012 0.4726564020922365
- link Link3: geometry collision box size=0.22858090290766803 0.8396552397938062 0.6279157854512294; visual box size=0.22858090290766803 0.8396552397938062 0.6279157854512294
- link Link4: geometry collision box size=0.7524356648259105 0.8007707306996854 0.3766565826450421; visual box size=0.7524356648259105 0.8007707306996854 0.3766565826450421
Joints:
- removed joint Link1_Link3
- removed joint Link2_Link4
- removed joint Link3_Link5
- removed joint Link3_Link6
- added joint Link2_Link3: type revolute, parent Link2, child Link3, origin xyz=-0.26872934650523495 0 0 rpy=0 0 0, axis 1 0 0, limit lower=-3.14159 upper=3.14159 effort=0.0 velocity=0.0
- added joint Link3_Link4: type revolute, parent Link3, child Link4, origin xyz=-0.11429045145383401 0 -0.3139578927256147 rpy=0 0 0, axis 1 0 0, limit lower=-3.14159 upper=3.14159 effort=0.0 velocity=0.0
- joint Link0_Link1: origin xyz=0 0 0.4397788389053114 rpy=0 0 0 -> xyz=0 0 0.2227436123548494 rpy=0 0 0
- joint Link1_Link2: origin xyz=0 0.4992171751666217 0.31796270810057414 rpy=0 0 0 -> xyz=-0.37515731827405174 0 0.4806772983597887 rpy=0 0 0
