Commit message: small color change

File: body0.urdf (robot description, URDF)
Before this commit: robot robot, 7 links, 6 joints
Links:
- link Link0: geometry collision box size=0.4256046756874421 0.40401650979552167 0.6008354066798793; visual box size=0.4256046756874421 0.40401650979552167 0.6008354066798793
- link Link1: geometry collision box size=0.3560754172206214 0.6144547811184597 0.33655072591889845; visual box size=0.3560754172206214 0.6144547811184597 0.33655072591889845
- link Link2: geometry collision box size=0.9815701708465605 0.5587942390559336 0.9071636185340217; visual box size=0.9815701708465605 0.5587942390559336 0.9071636185340217
- link Link3: geometry collision box size=0.8569193062973992 0.6754717366518134 0.42891927879210184; visual box size=0.8569193062973992 0.6754717366518134 0.42891927879210184
- link Link4: geometry collision box size=0.688134666339531 0.8651232744173785 0.9965855092542968; visual box size=0.688134666339531 0.8651232744173785 0.9965855092542968
- link Link5: geometry collision box size=0.7046157894024805 0.7589608706826911 0.4134002642002428; visual box size=0.7046157894024805 0.7589608706826911 0.4134002642002428
- link Link6: geometry collision box size=0.9993536364781406 0.2849408573069191 0.3502638025780249; visual box size=0.9993536364781406 0.2849408573069191 0.3502638025780249
Joints:
- removed joint Link0_Link3
- removed joint Link0_Link6
- removed joint Link1_Link4
- removed joint Link3_Link5
- added joint Link2_Link3: type revolute, parent Link2, child Link3, origin xyz=0 0 0.9071636185340217 rpy=0 0 0, axis 0 1 0, limit lower=-3.14159 upper=3.14159 effort=0.0 velocity=0.0
- added joint Link2_Link5: type revolute, parent Link2, child Link5, origin xyz=0 0.2793971195279668 0.45358180926701086 rpy=0 0 0, axis 0 0 1, limit lower=-3.14159 upper=3.14159 effort=0.0 velocity=0.0
- added joint Link3_Link4: type revolute, parent Link3, child Link4, origin xyz=0 0 0.42891927879210184 rpy=0 0 0, axis 1 0 0, limit lower=-3.14159 upper=3.14159 effort=0.0 velocity=0.0
- added joint Link4_Link6: type revolute, parent Link4, child Link6, origin xyz=0 0 0.9965855092542968 rpy=0 0 0, axis 0 1 0, limit lower=-3.14159 upper=3.14159 effort=0.0 velocity=0.0
- joint Link0_Link1: axis 0 0 1 -> 0 1 0; origin xyz=0.4423844117452832 0 0.30467850109868777 rpy=0 0 0 -> xyz=0.21280233784372105 0 0.30041770333993967 rpy=0 0 0
- joint Link0_Link2: axis 0 0 1 -> 1 0 0; origin xyz=0 0.4643556784540259 0.30467850109868777 rpy=0 0 0 -> xyz=0 0 0.6008354066798793 rpy=0 0 0

Commit message: rainbow colors

File: body0.urdf (robot description, URDF)
Before this commit: robot robot, 7 links, 6 joints
Links:
- link Link0: geometry collision box size=0.6091460522987651 0.7743941276618833 0.995293448925695; visual box size=0.6091460522987651 0.7743941276618833 0.995293448925695
- link Link1: geometry collision box size=0.9468022776416098 0.9938925218408365 0.46669434164408596; visual box size=0.9468022776416098 0.9938925218408365 0.46669434164408596
- link Link2: geometry collision box size=0.5698518365341583 0.3333770617482351 0.9383231775255554; visual box size=0.5698518365341583 0.3333770617482351 0.9383231775255554
- link Link3: geometry collision box size=0.23567860918506922 0.8497939962218597 0.4841227760072333; visual box size=0.23567860918506922 0.8497939962218597 0.4841227760072333
- link Link4: geometry collision box size=0.9925949693853686 0.4237765616362932 0.516562723465336; visual box size=0.9925949693853686 0.4237765616362932 0.516562723465336
- link Link5: geometry collision box size=0.6055486489209017 0.6280004407987941 0.533962739847534; visual box size=0.6055486489209017 0.6280004407987941 0.533962739847534
- link Link6: geometry collision box size=0.35277482474067723 0.3727742158021438 0.36291526060153906; visual box size=0.35277482474067723 0.3727742158021438 0.36291526060153906
Joints:
- removed joint Link2_Link5
- added joint Link0_Link5: type revolute, parent Link0, child Link5, origin xyz=0 -0.38719706383094166 0.4976467244628475 rpy=0 0 0, axis 1 0 0, limit lower=-3.14159 upper=3.14159 effort=0.0 velocity=0.0
- joint Link0_Link1: axis 0 1 0 -> 0 0 1; origin xyz=0.21280233784372105 0 0.30041770333993967 rpy=0 0 0 -> xyz=-0.30457302614938253 0 0.4976467244628475 rpy=0 0 0
- joint Link0_Link2: axis 1 0 0 -> 0 0 1; origin xyz=0 0 0.6008354066798793 rpy=0 0 0 -> xyz=0 0 0.995293448925695 rpy=0 0 0
- joint Link2_Link3: axis 0 1 0 -> 1 0 0; origin xyz=0 0 0.9071636185340217 rpy=0 0 0 -> xyz=-0.28492591826707914 0 0.4691615887627777 rpy=0 0 0
- joint Link3_Link4: axis 1 0 0 -> 0 1 0; origin xyz=0 0 0.42891927879210184 rpy=0 0 0 -> xyz=-0.11783930459253461 -0.42489699811092985 0 rpy=0 0 0
- joint Link4_Link6: axis 0 1 0 -> 0 0 1; origin xyz=0 0 0.9965855092542968 rpy=0 0 0 -> xyz=-0.4962974846926843 -0.2118882808181466 0 rpy=0 0 0

File: body1.urdf (robot description, URDF)
Before this commit: robot robot, 7 links, 6 joints
Links:
- link Link0: geometry collision box size=0.2063132390932827 0.4588637103130719 0.5393638054521832; visual box size=0.2063132390932827 0.4588637103130719 0.5393638054521832
- link Link1: geometry collision box size=0.27984998552686674 0.9208573310429522 0.32817685078512016; visual box size=0.27984998552686674 0.9208573310429522 0.32817685078512016
- link Link2: geometry collision box size=0.4877045645954084 0.7328256079282687 0.7712450292379851; visual box size=0.4877045645954084 0.7328256079282687 0.7712450292379851
- link Link3: geometry collision box size=0.5505017143502904 0.641136587365567 0.5102993310301813; visual box size=0.5505017143502904 0.641136587365567 0.5102993310301813
- link Link4: geometry collision box size=0.43577640326895284 0.29256671988446714 0.6509098630197641; visual box size=0.43577640326895284 0.29256671988446714 0.6509098630197641
- link Link5: geometry collision box size=0.4863392944205829 0.4802680428471835 0.9176104363509456; visual box size=0.4863392944205829 0.4802680428471835 0.9176104363509456
- link Link6: geometry collision box size=0.6615135266246384 0.672709616451479 0.5102904785350797; visual box size=0.6615135266246384 0.672709616451479 0.5102904785350797
Joints:
- removed joint Link0_Link3
- removed joint Link0_Link6
- removed joint Link1_Link4
- added joint Link2_Link3: type revolute, parent Link2, child Link3, origin xyz=0.2438522822977042 0 0.38562251461899255 rpy=0 0 0, axis 1 0 0, limit lower=-3.14159 upper=3.14159 effort=0.0 velocity=0.0
- added joint Link2_Link4: type revolute, parent Link2, child Link4, origin xyz=0 0 0.7712450292379851 rpy=0 0 0, axis 1 0 0, limit lower=-3.14159 upper=3.14159 effort=0.0 velocity=0.0
- added joint Link2_Link6: type revolute, parent Link2, child Link6, origin xyz=0 -0.36641280396413434 0.38562251461899255 rpy=0 0 0, axis 0 0 1, limit lower=-3.14159 upper=3.14159 effort=0.0 velocity=0.0
- joint Link0_Link1: axis 0 0 1 -> 0 1 0; origin xyz=0.4423844117452832 0 0.30467850109868777 rpy=0 0 0 -> xyz=-0.10315661954664135 0 0.2696819027260916 rpy=0 0 0
- joint Link0_Link2: axis 0 0 1 -> 1 0 0; origin xyz=0 0.4643556784540259 0.30467850109868777 rpy=0 0 0 -> xyz=0 0 0.5393638054521832 rpy=0 0 0
- joint Link3_Link5: origin xyz=0 -0.3246982140458653 0.21718229677407194 rpy=0 0 0 -> xyz=0.5505017143502904 0 0 rpy=0 0 0

Commit message: rectangular limbs

File: body0.urdf (robot description, URDF)
Before this commit: robot robot, 7 links, 6 joints
Links:
- link Link0: geometry collision box size=0.4438775463426045 0.5308984334481517 0.9630604060183654; visual box size=0.4438775463426045 0.5308984334481517 0.9630604060183654
- link Link1: geometry collision box size=0.4974131635250005 0.901633790194355 0.4110639207582578; visual box size=0.4974131635250005 0.901633790194355 0.4110639207582578
- link Link2: geometry collision box size=0.4326382523800254 0.7758337828495767 0.4463470659888713; visual box size=0.4326382523800254 0.7758337828495767 0.4463470659888713
- link Link3: geometry collision box size=0.824039973174475 0.2225618797846754 0.8919296661560345; visual box size=0.824039973174475 0.2225618797846754 0.8919296661560345
- link Link4: geometry collision box size=0.30867342099764955 0.9565378995104733 0.201891239737719; visual box size=0.30867342099764955 0.9565378995104733 0.201891239737719
- link Link5: geometry collision box size=0.9886125778522539 0.22113524522299496 0.2916398945642189; visual box size=0.9886125778522539 0.22113524522299496 0.2916398945642189
- link Link6: geometry collision box size=0.8653523377068784 0.3552483123579663 0.5623991683258902; visual box size=0.8653523377068784 0.3552483123579663 0.5623991683258902
Joints:
- removed joint Link0_Link2
- removed joint Link0_Link5
- removed joint Link2_Link3
- removed joint Link3_Link4
- removed joint Link4_Link6
- added joint Link0_Link3: type revolute, parent Link0, child Link3, origin xyz=0.22193877317130226 0 0.4815302030091827 rpy=0 0 0, axis 0 1 0, limit lower=-3.14159 upper=3.14159 effort=0.0 velocity=0.0
- added joint Link0_Link4: type revolute, parent Link0, child Link4, origin xyz=0 0 0.9630604060183654 rpy=0 0 0, axis 1 0 0, limit lower=-3.14159 upper=3.14159 effort=0.0 velocity=0.0
- added joint Link1_Link2: type revolute, parent Link1, child Link2, origin xyz=0.24870658176250024 0.4508168950971775 0 rpy=0 0 0, axis 0 0 1, limit lower=-3.14159 upper=3.14159 effort=0.0 velocity=0.0
- added joint Link3_Link5: type revolute, parent Link3, child Link5, origin xyz=0.824039973174475 0 0 rpy=0 0 0, axis 0 1 0, limit lower=-3.14159 upper=3.14159 effort=0.0 velocity=0.0
- added joint Link5_Link6: type revolute, parent Link5, child Link6, origin xyz=0.49430628892612694 0.11056762261149748 0 rpy=0 0 0, axis 0 1 0, limit lower=-3.14159 upper=3.14159 effort=0.0 velocity=0.0
- joint Link0_Link1: axis 0 0 1 -> 0 1 0; origin xyz=-0.30457302614938253 0 0.4976467244628475 rpy=0 0 0 -> xyz=0 0.26544921672407584 0.4815302030091827 rpy=0 0 0

File: body1.urdf (robot description, URDF)
Before this commit: robot robot, 7 links, 6 joints
Links:
- link Link0: geometry collision box size=0.4978258309485384 0.4478033514201856 0.613634977546186; visual box size=0.4978258309485384 0.4478033514201856 0.613634977546186
- link Link1: geometry collision box size=0.34205276265649176 0.9002867237729214 0.23890848970069922; visual box size=0.34205276265649176 0.9002867237729214 0.23890848970069922
- link Link2: geometry collision box size=0.2444047551299749 0.9618810758963416 0.3122232660849121; visual box size=0.2444047551299749 0.9618810758963416 0.3122232660849121
- link Link3: geometry collision box size=0.5388356496295637 0.6728203608745853 0.8600984075426747; visual box size=0.5388356496295637 0.6728203608745853 0.8600984075426747
- link Link4: geometry collision box size=0.335997403016605 0.9821542883784131 0.36916230425229; visual box size=0.335997403016605 0.9821542883784131 0.36916230425229
- link Link5: geometry collision box size=0.6127154549953638 0.9796288362063394 0.5283167591914335; visual box size=0.6127154549953638 0.9796288362063394 0.5283167591914335
- link Link6: geometry collision box size=0.7943755567274366 0.921799517163796 0.3033584595793688; visual box size=0.7943755567274366 0.921799517163796 0.3033584595793688
Joints:
- removed joint Link0_Link2
- removed joint Link2_Link4
- added joint Link1_Link2: type revolute, parent Link1, child Link2, origin xyz=0 -0.4501433618864607 0.11945424485034961 rpy=0 0 0, axis 0 1 0, limit lower=-3.14159 upper=3.14159 effort=0.0 velocity=0.0
- added joint Link3_Link4: type revolute, parent Link3, child Link4, origin xyz=0 0 0.8600984075426747 rpy=0 0 0, axis 0 0 1, limit lower=-3.14159 upper=3.14159 effort=0.0 velocity=0.0
- joint Link0_Link1: origin xyz=-0.10315661954664135 0 0.2696819027260916 rpy=0 0 0 -> xyz=0 0 0.613634977546186 rpy=0 0 0
- joint Link2_Link3: origin xyz=0.2438522822977042 0 0.38562251461899255 rpy=0 0 0 -> xyz=0 -0.4809405379481708 0.15611163304245604 rpy=0 0 0
- joint Link2_Link6: axis 0 0 1 -> 1 0 0; origin xyz=0 -0.36641280396413434 0.38562251461899255 rpy=0 0 0 -> xyz=-0.12220237756498745 -0.4809405379481708 0 rpy=0 0 0
- joint Link3_Link5: origin xyz=0.5505017143502904 0 0 rpy=0 0 0 -> xyz=-0.2694178248147818 0 0.4300492037713374 rpy=0 0 0
